Commit message: Fixed IK in gazebo

File: src/fmauch_universal_robot/ur_description/urdf/inc/ur5_macro.xacro (robot description, xacro)
@@ -75,5 +75,5 @@
   <parent link="tool"/>
   <child link="tooltip"/>
-  <origin xyz="0 -0.130 0.108" rpy="-0.157 0 0"/> <!-- the length of pen from center is 130mm -->
+  <origin xyz="0 -0.130 0.108" rpy="1.5707 0 3.1415"/> <!-- the length of pen from center is 130mm -->
 </joint>
    <xacro:include filename="$(find ur_description)/urdf/inc/ur_macro.xacro"/>
@@ -89,8 +89,20 @@
       safety_k_position="${safety_k_position}"
     />
+    <!--
+    <gazebo>
+      <plugin name="ros_control" filename="libgazebo_ros_control.so">
+        <robotNamespace>/</robotNamespace>
+        <robotSimtype>gazebo_ros_control/DefaultRobotHWSim</robotSimtype>
+      </plugin>
+    </gazebo>
+    -->
+        <!--
+      Inject Gazebo ROS Control plugin, which allows us to use ros_control
+      controllers to control the virtual robot hw.
+    -->
     <gazebo>
       <plugin name="ros_control" filename="libgazebo_ros_control.so">
         <!--robotNamespace>/</robotNamespace-->
-        <!--robotSimtype>gazebo_ros_control/DefaultRobotHWSim</robotSimtype-->
+        <!--robotSimType>gazebo_ros_control/DefaultRobotHWSim</robotSimType-->
       </plugin>
     </gazebo>

Commit message: Tested code on real robot

File: src/fmauch_universal_robot/ur_description/urdf/inc/ur5_macro.xacro (robot description, xacro)
@@ -75,5 +75,5 @@
   <parent link="tool"/>
   <child link="tooltip"/>
-  <origin xyz="0 -0.130 0.108" rpy="1.5707 0 3.1415"/> <!-- the length of pen from center is 130mm -->
+  <origin xyz="0 -0.130 0.108" rpy="1.5707 0 3.4906"/> <!-- the length of pen from center is 130mm -->
 </joint>
    <xacro:include filename="$(find ur_description)/urdf/inc/ur_macro.xacro"/>
